Commit message: Minesweepers work + Launch Rviz along Gazebo

File: GoChaseIt_ws/src/my_robot/urdf/my_robot.xacro (robot description, xacro)
@@ -1,4 +1,5 @@
 <?xml version='1.0'?>
 <robot name="my_robot" xmlns:xacro="http://www.ros.org/wiki/xacro">
+  <xacro:include filename="$(find my_robot)/urdf/my_robot.gazebo" />
   <link name="robot_footprint"></link>
   <joint name="robot_footprint_joint" type="fixed">
@@ -76,13 +77,13 @@
         <cylinder radius="0.05" length="0.025"/>
       </geometry>
-      <material name="">
-        <color rgba="1 0.3 0.4 1"/>
-      </material>
-    </collision>
-    <visual name='wheel_visual'>
-      <origin xyz="0 0 0" rpy=" 0 1.5707 1.5707"/>
-      <geometry>
-        <cylinder radius="0.05" length="0.025"/>
-      </geometry>
+    </collision>
+    <visual name='wheel_visual'>
+      <origin xyz="0 0 0" rpy=" 0 1.5707 1.5707"/>
+      <geometry>
+        <cylinder radius="0.05" length="0.025"/>
+      </geometry>
+      <!-- <material name="-">
+        <color rgba="1 0.3 0.4 1"/>
+      </material> -->
     </visual>
   </link>
@@ -102,13 +103,13 @@
         <cylinder radius="0.05" length="0.025"/>
       </geometry>
-      <material name="">
-        <color rgba="1 0.3 0.4 1"/>
-      </material>
-    </collision>
-    <visual name='wheel_visual'>
-      <origin xyz="0 0 0" rpy=" 0 1.5707 1.5707"/>
-      <geometry>
-        <cylinder radius="0.05" length="0.025"/>
-      </geometry>
+    </collision>
+    <visual name='wheel_visual'>
+      <origin xyz="0 0 0" rpy=" 0 1.5707 1.5707"/>
+      <geometry>
+        <cylinder radius="0.05" length="0.025"/>
+      </geometry>
+      <!-- <material name="">
+        <color rgba="1 0.3 0.4 1"/>
+      </material> -->
     </visual>
   </link>
@@ -134,7 +135,7 @@
         <cylinder radius="0.05" length="0.025"/>
       </geometry>
-      <material name="">
-        <color rgba="1 0.3 0.4 1"/>
-      </material>
+      <!-- <material name="">
+        <color rgba="1 0.3 0.4 1"/>
+      </material> -->
     </visual>
   </link>
@@ -160,9 +161,15 @@
         <cylinder radius="0.05" length="0.025"/>
       </geometry>
-      <material name="">
-        <color rgba="1 0.3 0.4 1"/>
-      </material>
-    </visual>
-  </link>
+      <!-- <material name="">
+        <color rgba="1 0.3 0.4 1"/>
+      </material> -->
+    </visual>
+  </link>
+  <gazebo reference="chassis">
+    <material>
+      Gazebo/Orange
+        <!-- <color rgba="0 1 0 1"/> -->
+    </material>
+  </gazebo>
   <joint type="continuous" name="front_right_wheel_hinge">
     <origin xyz="0.15 0.12 -0.05" rpy="0 0 0"/>
@@ -197,3 +204,69 @@
     <dynamics damping="1.0" friction="1.0"/>
   </joint>
+  <!-- Camera link-->
+  <link name="camera">
+    <inertial>
+      <mass value="0.1"/>
+      <origin xyz=".05 .05 .05" rpy="0 0 0"/>
+      <inertia
+          ixx="1e-6" ixy="0" ixz="0"
+          iyy="1e-6" iyz="0"
+          izz="1e-6"
+      />
+    </inertial>
+    <collision name='collision'>
+      <origin xyz="0 0 0" rpy=" 0 0 0"/>
+      <geometry>
+        <box size=".05 .05 .05"/>
+      </geometry>
+    </collision>
+    <visual name='camera_visual'>
+      <origin xyz="0 0 0" rpy=" 0 0 0"/>
+      <geometry>
+        <box size=".05 .05 .05"/>
+      </geometry>
+    </visual>
+  </link>
+  <!-- Camera joint -->
+  <joint type="fixed" name="camera_joint">
+    <origin xyz="0.2 0 0" rpy="0 0 0"/>
+    <child link="camera"/>
+    <parent link="chassis"/>
+    <axis xyz="0 1 0" rpy="0 0 0"/>
+    <limit effort="10000" velocity="1000"/>
+    <dynamics damping="1.0" friction="1.0"/>
+  </joint>
+  <!-- Hokuyo lidar sensor -->
+  <link name="hokuyo">
+    <inertial>
+      <mass value="1e-5"/>
+      <origin xyz="0 0 0" rpy=" 0 0 0"/>
+      <inertia
+          ixx="1e-6" ixy="0" ixz="0"
+          iyy="1e-6" iyz="0"
+          izz="1e-6"
+      />
+    </inertial>
+    <collision name='collision'>
+      <origin xyz="0 0 0" rpy=" 0 0 0"/>
+      <geometry>
+        <mesh filename="package://my_robot/meshes/hokuyo.dae"/>
+      </geometry>
+    </collision>
+    <visual name='hokuyo_visual'>
+      <origin xyz="0 0 0" rpy=" 0 0 0"/>
+      <geometry>
+        <mesh filename="package://my_robot/meshes/hokuyo.dae"/>
+      </geometry>
+    </visual>
+  </link>
+  <!-- hokuyo joint -->
+  <joint type="fixed" name="hokuyo_joint">
+    <origin xyz="0.15 0 0.1" rpy="0 0 0"/>
+    <child link="hokuyo"/>
+    <parent link="chassis"/>
+    <axis xyz="0 1 0" rpy="0 0 0"/>
+    <limit effort="10000" velocity="1000"/>
+    <dynamics damping="1.0" friction="1.0"/>
+  </joint>
 </robot>

Commit message: img.step not img.hight

File: GoChaseIt_ws/src/my_robot/urdf/my_robot.xacro (robot description, xacro)
@@ -31,5 +31,5 @@
       </geometry>
     </visual>
-    <!-- <collision name='back_caster_collision'>
+    <collision name='back_caster_collision'>
       <origin xyz="-0.15 0 -0.05" rpy=" 0 0 0"/>
       <geometry>
@@ -42,7 +42,4 @@
         <sphere radius="0.05"/>
       </geometry>
-      <material name="">
-        <color rgba="1 37/255 229/255 0.8"/>
-      </material>
     </visual>
     <collision name='front_caster_collision'>
@@ -57,35 +54,29 @@
         <sphere radius="0.05"/>
       </geometry>
-     <material name="">
-        <color rgba="1 37/255 229/255 0.8"/>
-      </material>
-    </visual> -->
-  </link>
-  <link name="back_right_wheel">
-    <inertial>
-      <mass value="5.0"/>
-      <origin xyz="0 0 0" rpy=" 0 1.5707 1.5707"/>
-      <inertia
-          ixx="0.1" ixy="0" ixz="0"
-          iyy="0.1" iyz="0"
-          izz="0.1"
-      />
-    </inertial>
-    <collision name='collision'>
-      <origin xyz="0 0 0" rpy=" 0 1.5707 1.5707"/>
-      <geometry>
-        <cylinder radius="0.05" length="0.025"/>
-      </geometry>
-    </collision>
-    <visual name='wheel_visual'>
-      <origin xyz="0 0 0" rpy=" 0 1.5707 1.5707"/>
-      <geometry>
-        <cylinder radius="0.05" length="0.025"/>
-      </geometry>
-      <!-- <material name="-">
-        <color rgba="1 0.3 0.4 1"/>
-      </material> -->
-    </visual>
-  </link>
+    </visual>
+  </link>
+  <!-- <link name="back_right_wheel">
+    <inertial>
+      <mass value="5.0"/>
+      <origin xyz="0 0 0" rpy=" 0 1.5707 1.5707"/>
+      <inertia
+          ixx="0.1" ixy="0" ixz="0"
+          iyy="0.1" iyz="0"
+          izz="0.1"
+      />
+    </inertial>
+    <collision name='collision'>
+      <origin xyz="0 0 0" rpy=" 0 1.5707 1.5707"/>
+      <geometry>
+        <cylinder radius="0.05" length="0.025"/>
+      </geometry>
+    </collision>
+    <visual name='wheel_visual'>
+      <origin xyz="0 0 0" rpy=" 0 1.5707 1.5707"/>
+      <geometry>
+        <cylinder radius="0.05" length="0.025"/>
+      </geometry>
+    </visual>
+  </link> -->
   <link name="front_right_wheel">
     <inertial>
@@ -109,35 +100,29 @@
         <cylinder radius="0.05" length="0.025"/>
       </geometry>
-      <!-- <material name="">
-        <color rgba="1 0.3 0.4 1"/>
-      </material> -->
-    </visual>
-  </link>
-  <link name="back_left_wheel">
-    <inertial>
-      <mass value="5.0"/>
-      <origin xyz="0 0 0" rpy=" 0 1.5707 1.5707"/>
-      <inertia
-          ixx="0.1" ixy="0" ixz="0"
-          iyy="0.1" iyz="0"
-          izz="0.1"
-      />
-    </inertial>
-    <collision name='collision'>
-      <origin xyz="0 0 0" rpy=" 0 1.5707 1.5707"/>
-      <geometry>
-        <cylinder radius="0.05" length="0.025"/>
-      </geometry>
-    </collision>
-    <visual name='wheel_visual'>
-      <origin xyz="0 0 0" rpy=" 0 1.5707 1.5707"/>
-      <geometry>
-        <cylinder radius="0.05" length="0.025"/>
-      </geometry>
-      <!-- <material name="">
-        <color rgba="1 0.3 0.4 1"/>
-      </material> -->
-    </visual>
-  </link>
+    </visual>
+  </link>
+  <!-- <link name="back_left_wheel">
+    <inertial>
+      <mass value="5.0"/>
+      <origin xyz="0 0 0" rpy=" 0 1.5707 1.5707"/>
+      <inertia
+          ixx="0.1" ixy="0" ixz="0"
+          iyy="0.1" iyz="0"
+          izz="0.1"
+      />
+    </inertial>
+    <collision name='collision'>
+      <origin xyz="0 0 0" rpy=" 0 1.5707 1.5707"/>
+      <geometry>
+        <cylinder radius="0.05" length="0.025"/>
+      </geometry>
+    </collision>
+    <visual name='wheel_visual'>
+      <origin xyz="0 0 0" rpy=" 0 1.5707 1.5707"/>
+      <geometry>
+        <cylinder radius="0.05" length="0.025"/>
+      </geometry>
+    </visual>
+  </link> -->
   <link name="front_left_wheel">
     <inertial>
@@ -161,7 +146,4 @@
         <cylinder radius="0.05" length="0.025"/>
       </geometry>
-      <!-- <material name="">
-        <color rgba="1 0.3 0.4 1"/>
-      </material> -->
     </visual>
   </link>
@@ -173,5 +155,5 @@
   </gazebo>
   <joint type="continuous" name="front_right_wheel_hinge">
-    <origin xyz="0.15 0.12 -0.05" rpy="0 0 0"/>
+    <origin xyz="0 0.12 -0.05" rpy="0 0 0"/>
     <child link="front_right_wheel"/>
     <parent link="chassis"/>
@@ -180,5 +162,5 @@
     <dynamics damping="1.0" friction="1.0"/>
   </joint>
-  <joint type="continuous" name="back_right_wheel_hinge">
+  <!-- <joint type="continuous" name="back_right_wheel_hinge">
     <origin xyz="-0.15 0.12 -0.05" rpy="0 0 0"/>
     <child link="back_right_wheel"/>
@@ -187,7 +169,7 @@
     <limit effort="10000" velocity="1000"/>
     <dynamics damping="1.0" friction="1.0"/>
-  </joint>
+  </joint> -->
     <joint type="continuous" name="front_left_wheel_hinge">
-    <origin xyz="0.15 -0.12 -0.05" rpy="0 0 0"/>
+    <origin xyz="0 -0.12 -0.05" rpy="0 0 0"/>
     <child link="front_left_wheel"/>
     <parent link="chassis"/>
@@ -196,4 +178,5 @@
     <dynamics damping="1.0" friction="1.0"/>
   </joint>
+<!--
   <joint type="continuous" name="back_left_wheel_hinge">
     <origin xyz="-0.15 -0.12 -0.05" rpy="0 0 0"/>
@@ -203,5 +186,5 @@
     <limit effort="10000" velocity="1000"/>
     <dynamics damping="1.0" friction="1.0"/>
-  </joint>
+  </joint> -->
   <!-- Camera link-->
   <link name="camera">
